Commit message: Drop asus_xtion_pro_offset.urdf.xacro and use instead a parameterised asus_xtion_pro.urdf.xacro (#280)
Also drop asus_ from camera name, to match the other cameras that don't include the manufacturer

File: turtlebot_description/robots/create_circles_asus_xtion_pro.urdf.xacro (robot description, xacro)
@@ -9,7 +9,7 @@
   <xacro:include filename="$(find create_description)/urdf/create.urdf.xacro"/>
   <xacro:include filename="$(find turtlebot_description)/urdf/stacks/circles.urdf.xacro"/>
-  <xacro:include filename="$(find turtlebot_description)/urdf/sensors/asus_xtion_pro.urdf.xacro"/>
+  <xacro:include filename="$(find turtlebot_description)/urdf/sensors/xtion_pro.urdf.xacro"/>
   <xacro:create/>
-  <xacro:stack_circles parent="base_link"/>
-  <xacro:sensor_asus_xtion_pro  parent="base_link"/>
+  <xacro:stack_circles    parent="base_link"/>
+  <xacro:sensor_xtion_pro parent="base_link"/>
 </robot>

File: turtlebot_description/robots/create_circles_kinect.urdf.xacro (robot description, xacro)
@@ -12,4 +12,4 @@
   <xacro:create/>
   <xacro:stack_circles parent="base_link"/>
-  <xacro:sensor_kinect  parent="base_link"/>
+  <xacro:sensor_kinect parent="base_link"/>
 </robot>

File: turtlebot_description/robots/kobuki_hexagons_astra.urdf.xacro (robot description, xacro)
@@ -12,4 +12,4 @@
   <xacro:kobuki/>
   <xacro:stack_hexagons parent="base_link"/>
-  <xacro:sensor_astra parent="base_link"/>
+  <xacro:sensor_astra   parent="base_link"/>
 </robot>

File: turtlebot_description/robots/kobuki_hexagons_asus_xtion_pro.urdf.xacro (robot description, xacro)
@@ -9,7 +9,7 @@
   <xacro:include filename="$(find kobuki_description)/urdf/kobuki.urdf.xacro" />
   <xacro:include filename="$(find turtlebot_description)/urdf/stacks/hexagons.urdf.xacro"/>
-  <xacro:include filename="$(find turtlebot_description)/urdf/sensors/asus_xtion_pro.urdf.xacro"/>
+  <xacro:include filename="$(find turtlebot_description)/urdf/sensors/xtion_pro.urdf.xacro"/>
   <xacro:kobuki/>
-  <xacro:stack_hexagons                 parent="base_link"/>
-  <xacro:sensor_asus_xtion_pro          parent="base_link"/>
+  <xacro:stack_hexagons   parent="base_link"/>
+  <xacro:sensor_xtion_pro parent="base_link" xtion_pro_cam_py="0.0205"/>
 </robot>

File: turtlebot_description/robots/kobuki_hexagons_asus_xtion_pro_offset.urdf.xacro (robot description, xacro)
@@ -9,7 +9,7 @@
   <xacro:include filename="$(find kobuki_description)/urdf/kobuki.urdf.xacro" />
   <xacro:include filename="$(find turtlebot_description)/urdf/stacks/hexagons.urdf.xacro"/>
-  <xacro:include filename="$(find turtlebot_description)/urdf/sensors/asus_xtion_pro_offset.urdf.xacro"/>
+  <xacro:include filename="$(find turtlebot_description)/urdf/sensors/xtion_pro.urdf.xacro"/>
   <xacro:kobuki/>
-  <xacro:stack_hexagons                 parent="base_link"/>
-  <xacro:sensor_asus_xtion_pro_offset   parent="base_link"/>
+  <xacro:stack_hexagons   parent="base_link"/>
+  <xacro:sensor_xtion_pro parent="base_link" xtion_pro_cam_py="-0.0125"/>
 </robot>

File: turtlebot_description/robots/kobuki_hexagons_kinect.urdf.xacro (robot description, xacro)
@@ -12,4 +12,4 @@
   <xacro:kobuki/>
   <xacro:stack_hexagons parent="base_link"/>
-  <xacro:sensor_kinect  parent="base_link"/>
+  <xacro:sensor_kinect parent="base_link"/>
 </robot>

File: turtlebot_description/robots/kobuki_hexagons_r200.urdf.xacro (robot description, xacro)
@@ -12,4 +12,4 @@
   <xacro:kobuki/>
   <xacro:stack_hexagons parent="base_link"/>
-  <xacro:sensor_r200  parent="base_link"/>
+  <xacro:sensor_r200    parent="base_link"/>
 </robot>

File: turtlebot_description/urdf/sensors/xtion_pro.urdf.xacro (robot description, xacro)
@@ -1,14 +1,14 @@
 <?xml version="1.0"?>
-<robot name="sensor_asus_xtion_pro" xmlns:xacro="http://ros.org/wiki/xacro">
+<robot name="sensor_xtion_pro" xmlns:xacro="http://ros.org/wiki/xacro">
   <xacro:include filename="$(find turtlebot_description)/urdf/turtlebot_gazebo.urdf.xacro"/>
   <xacro:include filename="$(find turtlebot_description)/urdf/turtlebot_properties.urdf.xacro"/>
   <!-- Xacro properties -->
-  <xacro:property name="asus_xtion_pro_cam_py" value="0.0205"/>
-  <xacro:property name="asus_xtion_pro_depth_rel_rgb_py" value="0.0270" />
-  <xacro:property name="asus_xtion_pro_cam_rel_rgb_py"   value="-0.0220" />
+  <xacro:property name="xtion_pro_depth_rel_rgb_py" value="0.0270" />
+  <xacro:property name="xtion_pro_cam_rel_rgb_py"   value="-0.0220" />
   <!-- Parameterised in part by the values in turtlebot_properties.urdf.xacro -->
-  <xacro:macro name="sensor_asus_xtion_pro" params="parent">
+  <!-- xtion_pro_cam_py allows for a camera displaced so the depth optical frame aligns with robot center -->
+  <xacro:macro name="sensor_xtion_pro" params="parent xtion_pro_cam_py">
     <joint name="camera_rgb_joint" type="fixed">
-      <origin xyz="${cam_px} ${asus_xtion_pro_cam_py} ${cam_pz}"
+      <origin xyz="${cam_px} ${xtion_pro_cam_py} ${cam_pz}"
               rpy="${cam_or} ${cam_op} ${cam_oy}"/>
       <parent link="${parent}"/>
@@ -23,5 +23,5 @@
     <link name="camera_rgb_optical_frame"/>
     <joint name="camera_joint" type="fixed">
-      <origin xyz="0 ${asus_xtion_pro_cam_rel_rgb_py} 0"
+      <origin xyz="0 ${xtion_pro_cam_rel_rgb_py} 0"
               rpy="0 0 0"/>
       <parent link="camera_rgb_frame"/>
@@ -50,5 +50,5 @@
     </link>
     <joint name="camera_depth_joint" type="fixed">
-      <origin xyz="0 ${asus_xtion_pro_depth_rel_rgb_py} 0" rpy="0 0 0" />
+      <origin xyz="0 ${xtion_pro_depth_rel_rgb_py} 0" rpy="0 0 0" />
       <parent link="camera_rgb_frame" />
       <child link="camera_depth_frame" />
@@ -64,10 +64,10 @@
     <xacro:turtlebot_sim_3dsensor/>
     <!-- Asus mount -->
-    <joint name="mount_asus_xtion_pro_joint" type="fixed">
+    <joint name="mount_xtion_pro_joint" type="fixed">
       <origin xyz="-0.1024 0.0 0.272" rpy="0 0 0"/>
       <parent link="${parent}"/>
-      <child link="mount_asus_xtion_pro_link"/>
+      <child link="mount_xtion_pro_link"/>
     </joint>
-    <link name="mount_asus_xtion_pro_link">
+    <link name="mount_xtion_pro_link">
       <visual>
         <origin xyz="0 0 0" rpy="${-M_PI/2} 0 0"/>
