Commit message: Replace the cylinder collision model of top and middle plates with a simplified mesh

File: turtlebot_description/urdf/stacks/hexagons.urdf.xacro (robot description, xacro)
@@ -178,5 +178,6 @@
         <origin xyz="0.01364 0.0 0.0" rpy="0 0 0"/>
         <geometry>
-          <cylinder length="0.006" radius="0.170"/>
+          <mesh filename="package://turtlebot_description/meshes/stacks/hexagons/plate_simple.stl"
+                scale="${M_SCALE} ${M_SCALE} ${M_SCALE}"/>
         </geometry>
       </collision>
@@ -210,5 +211,6 @@
         <origin xyz="0.01364 0 0" rpy="0 0 0"/>
         <geometry>
-          <cylinder length="0.006" radius="0.170"/>
+          <mesh filename="package://turtlebot_description/meshes/stacks/hexagons/plate_simple.stl"
+                scale="${M_SCALE} ${M_SCALE} ${M_SCALE}"/>
         </geometry>
       </collision>

Commit message: Add optional euler angles to pole macros (no effect by default)

File: turtlebot_description/urdf/stacks/hexagons.urdf.xacro (robot description, xacro)
@@ -9,7 +9,7 @@
   <!-- Xacro macros -->
   <!-- Pole macros -->
-  <xacro:macro name="stack_bottom_pole" params="parent number x_loc y_loc z_loc">
+  <xacro:macro name="stack_bottom_pole" params="parent number x_loc y_loc z_loc roll=0.0 pitch=0.0 yaw=0.0">
     <joint name="pole_bottom_${number}_joint" type="fixed">
-      <origin xyz="${x_loc} ${y_loc} ${z_loc}" rpy="0 0 0"/>
+      <origin xyz="${x_loc} ${y_loc} ${z_loc}" rpy="${roll} ${pitch} ${yaw}"/>
       <parent link="${parent}"/>
       <child link="pole_bottom_${number}_link"/>
@@ -37,7 +37,7 @@
     </link>
   </xacro:macro>
-  <xacro:macro name="stack_middle_pole" params="parent number x_loc y_loc z_loc">
+  <xacro:macro name="stack_middle_pole" params="parent number x_loc y_loc z_loc roll=0.0 pitch=0.0 yaw=0.0">
     <joint name="pole_middle_${number}_joint" type="fixed">
-      <origin xyz="${x_loc} ${y_loc} ${z_loc}" rpy="0 0 0" />
+      <origin xyz="${x_loc} ${y_loc} ${z_loc}" rpy="${roll} ${pitch} ${yaw}" />
       <parent link="${parent}"/>
       <child link="pole_middle_${number}_link"/>
@@ -65,7 +65,7 @@
     </link>
   </xacro:macro>
-  <xacro:macro name="stack_top_pole" params="parent number x_loc y_loc z_loc">
+  <xacro:macro name="stack_top_pole" params="parent number x_loc y_loc z_loc roll=0.0 pitch=0.0 yaw=0.0">
     <joint name="pole_top_${number}_joint" type="fixed">
-      <origin xyz="${x_loc} ${y_loc} ${z_loc}" rpy="0 0 0"/>
+      <origin xyz="${x_loc} ${y_loc} ${z_loc}" rpy="${roll} ${pitch} ${yaw}"/>
       <parent link="${parent}"/>
       <child link="pole_top_${number}_link"/>
@@ -93,7 +93,7 @@
     </link>
   </xacro:macro>
-  <xacro:macro name="stack_3d_sensor_pole" params="parent number x_loc y_loc z_loc">
+  <xacro:macro name="stack_3d_sensor_pole" params="parent number x_loc y_loc z_loc roll=0.0 pitch=0.0 yaw=0.0">
     <joint name="pole_kinect_${number}_joint" type="fixed">
-      <origin xyz="${x_loc} ${y_loc} ${z_loc}" rpy="0 0 0"/>
+      <origin xyz="${x_loc} ${y_loc} ${z_loc}" rpy="${roll} ${pitch} ${yaw}"/>
       <parent link="${parent}"/>
       <child link="pole_kinect_${number}_link"/>
